Commit message: refined manipulability calc using quaternions and added in an arc oriented away from the prune point for better manipulability

File: urdf/rpr_manipulator.urdf (robot description, URDF)
Before this commit: robot rpr_manipulator, 8 links, 7 joints
Joints:
- joint joint4: origin xyz=0 0 0.025 rpy=0 0 0 -> xyz=0 0 0.025 rpy=0 0 1.57

File: urdf/rrr_manipulator.urdf (robot description, URDF)
Before this commit: robot rrr_manipulator, 8 links, 7 joints
Joints:
- joint joint4: origin xyz=0 0 0.025 rpy=0 0 0 -> xyz=0 0 0.025 rpy=0 0 1.57
