Commit message: created new 4dof urdfs. condensed testing code into main script

File: urdf/rprr_manipulator.urdf (robot description, URDF)
Before this commit: robot prrr_manipulator, 9 links, 8 joints
Joints:
- joint prismatic1: axis 0 1 0 -> 0 0 1; origin xyz=0 0 0.125 rpy=0 0 0 -> xyz=0 0 0.005 rpy=0 0 0; parent base_link -> link2
- joint revolute1: origin xyz=0 0 0 rpy=0 0 0 -> xyz=0 0 0.125 rpy=0 0 0; parent prismatic_link -> base_link
- joint revolute2: parent link2 -> prismatic_link

File: urdf/rrpr_manipulator.urdf (robot description, URDF)
Before this commit: robot prrr_manipulator, 9 links, 8 joints
Joints:
- joint prismatic1: origin xyz=0 0 0.125 rpy=0 0 0 -> xyz=0 0 0.005 rpy=0 0 0; parent base_link -> link3
- joint revolute1: origin xyz=0 0 0 rpy=0 0 0 -> xyz=0 0 0.125 rpy=0 0 0; parent prismatic_link -> base_link
- joint revolute3: parent link3 -> prismatic_link

File: urdf/rrrp_manipulator.urdf (robot description, URDF)
Before this commit: robot prrr_manipulator, 9 links, 8 joints
Joints:
- joint fixed1: parent link4 -> prismatic_link
- joint prismatic1: origin xyz=0 0 0.125 rpy=0 0 0 -> xyz=0 0 0.005 rpy=0 0 0; parent base_link -> link4
- joint revolute1: origin xyz=0 0 0 rpy=0 0 0 -> xyz=0 0 0.125 rpy=0 0 0; parent prismatic_link -> base_link
