Commit message: plotting for arc manipulability, condesing code for readability, adjusting manipulability calculation for planar system

File: urdf/prrr_manipulator.urdf (robot description, URDF)
Before this commit: robot six_dof_manipulator_with_gripper, 10 links, 9 joints
Links:
- removed link link5
- link link1: geometry 
Joints:
- removed joint joint1
- removed joint joint2
- removed joint joint3
- removed joint joint4
- removed joint joint5
- removed joint joint6
- removed joint joint7
- removed joint joint8
- removed joint joint9
- added joint fixed1: type fixed, parent link4, child wrist, origin xyz=0 0 0.525 rpy=0 0 1.57, axis 0 0 1, limit lower=-3.14 upper=3.14 effort=10 velocity=1
- added joint fixed2: type fixed, parent wrist, child left_finger, origin xyz=-0.1 0 0.075 rpy=0 0 0
- added joint fixed3: type fixed, parent wrist, child right_finger, origin xyz=0.1 0 0.075 rpy=0 0 0
- added joint fixed4: type fixed, parent wrist, child gripper_center, origin xyz=0 0 0.15 rpy=0 0 0
- added joint prismatic1: type prismatic, parent base_link, child link1, origin xyz=0 0 0.125 rpy=0 0 0, axis 0 1 0, limit lower=-0.5 upper=0.5 effort=10 velocity=1
- added joint revolute1: type revolute, parent link1, child link2, origin xyz=0 0 0 rpy=0 0 0, axis 1 0 0, limit lower=-3.14 upper=3.14 effort=10 velocity=1
- added joint revolute2: type revolute, parent link2, child link3, origin xyz=0 0 0.5 rpy=0 0 0, axis 1 0 0, limit lower=-3.14 upper=3.14 effort=10 velocity=1
- added joint revolute3: type revolute, parent link3, child link4, origin xyz=0 0 0.5 rpy=0 0 0, axis 1 0 0, limit lower=-3.14 upper=3.14 effort=10 velocity=1

File: urdf/rrr_manipulator.urdf (robot description, URDF)
Before this commit: robot rrr_manipulator, 8 links, 7 joints
Links:
- link left_finger: geometry collision box size=0.05 0.05 0.15; visual box size=0.05 0.05 0.15
- link right_finger: geometry collision box size=0.05 0.05 0.15; visual box size=0.05 0.05 0.15
Joints:
- joint joint4: axis (none) -> 0 0 1; limit (none) -> lower=-3.14 upper=3.14 effort=10 velocity=1; origin xyz=0 0 0.025 rpy=0 0 1.57 -> xyz=0 0 0.525 rpy=0 0 1.57
- joint joint5: origin xyz=-0.1 0 0.15 rpy=0 0 0 -> xyz=-0.1 0 0.075 rpy=0 0 0
- joint joint6: origin xyz=0.1 0 0.65 rpy=0 0 0 -> xyz=0.1 0 0.075 rpy=0 0 0
- joint joint7: origin xyz=0 0 0.7 rpy=0 0 0 -> xyz=0 0 0.15 rpy=0 0 0

Commit message: generate an rrr_manipulator using element tree. updated gripper wrist rotation

File: urdf/prrr_manipulator.urdf (robot description, URDF)
Before this commit: robot prrr_manipulator, 9 links, 8 joints
Links:
- link wrist: geometry collision box size=0.05 0.25 0.05; visual box size=0.05 0.25 0.05
Joints:
- joint fixed1: origin xyz=0 0 0.525 rpy=0 0 1.57 -> xyz=0 0 0.525 rpy=0 0 0
- joint fixed2: origin xyz=-0.1 0 0.075 rpy=0 0 0 -> xyz=0 -0.1 0.075 rpy=0 0 0
- joint fixed3: origin xyz=0.1 0 0.075 rpy=0 0 0 -> xyz=0 0.1 0.075 rpy=0 0 0

File: urdf/rprr_manipulator.urdf (robot description, URDF)
Before this commit: robot prrr_manipulator, 9 links, 8 joints
Links:
- link link2: geometry visual cylinder length=0.5 radius=0.05
- link link3: geometry visual cylinder length=0.5 radius=0.05
- link wrist: geometry collision box size=0.05 0.25 0.05; visual box size=0.05 0.25 0.05
Joints:
- joint fixed1: origin xyz=0 0 0.525 rpy=0 0 1.57 -> xyz=0 0 0.525 rpy=0 0 0
- joint fixed2: origin xyz=-0.1 0 0.075 rpy=0 0 0 -> xyz=0 -0.1 0.075 rpy=0 0 0
- joint fixed3: origin xyz=0.1 0 0.075 rpy=0 0 0 -> xyz=0 0.1 0.075 rpy=0 0 0

File: urdf/rrpr_manipulator.urdf (robot description, URDF)
Before this commit: robot prrr_manipulator, 9 links, 8 joints
Links:
- link wrist: geometry collision box size=0.05 0.25 0.05; visual box size=0.05 0.25 0.05
Joints:
- joint fixed1: origin xyz=0 0 0.525 rpy=0 0 1.57 -> xyz=0 0 0.525 rpy=0 0 0
- joint fixed2: origin xyz=-0.1 0 0.075 rpy=0 0 0 -> xyz=0 -0.1 0.075 rpy=0 0 0
- joint fixed3: origin xyz=0.1 0 0.075 rpy=0 0 0 -> xyz=0 0.1 0.075 rpy=0 0 0

File: urdf/rrr_manipulator.urdf (robot description, URDF)
Before this commit: robot rrr_manipulator, 8 links, 7 joints
Links:
- link wrist: geometry collision box size=0.05 0.25 0.05; visual box size=0.05 0.25 0.05
Joints:
- joint joint4: origin xyz=0 0 0.525 rpy=0 0 1.57 -> xyz=0 0 0.525 rpy=0 0 0
- joint joint5: origin xyz=-0.1 0 0.075 rpy=0 0 0 -> xyz=0 -0.1 0.075 rpy=0 0 0
- joint joint6: origin xyz=0.1 0 0.075 rpy=0 0 0 -> xyz=0 0.1 0.075 rpy=0 0 0

File: urdf/rrrp_manipulator.urdf (robot description, URDF)
Before this commit: robot prrr_manipulator, 9 links, 8 joints
Links:
- link link4: geometry visual cylinder length=0.5 radius=0.05
- link wrist: geometry visual box size=0.05 0.25 0.05
Joints:
- joint fixed1: origin xyz=0 0 0.525 rpy=0 0 1.57 -> xyz=0 0 0.525 rpy=0 0 0
- joint fixed2: origin xyz=-0.1 0 0.075 rpy=0 0 0 -> xyz=0 -0.1 0.075 rpy=0 0 0
- joint fixed3: origin xyz=0.1 0 0.075 rpy=0 0 0 -> xyz=0 0.1 0.075 rpy=0 0 0
- joint prismatic1: axis 0 1 0 -> 0 0 1
