Commit message: refactoring to isolate pybullet and point sampling functionality

File: urdf/ur5e/ur5e_cart.urdf (robot description, URDF)
Before this commit: robot ur5e, 15 links, 14 joints
Joints:
- joint mount_base_joint: origin xyz=0.0 0.0 0.0 rpy=0.0 0.0 -1.5708 -> xyz=0.0 0.0 0.0 rpy=0.0 0.0 2.35

Commit message: adjusted ur5 home config. verified path interpolation

File: urdf/ur5e/ur5e_cart.urdf (robot description, URDF)
Before this commit: robot ur5e, 15 links, 14 joints
Joints:
- joint elbow_joint: origin xyz=-0.425282422158 0 0 rpy=3.14087106174 3.14130791395 -3.1415908958 -> xyz=-0.425282422158 0 0 rpy=3.14087106174 3.14130791395 -1.047
- joint shoulder_lift_joint: origin xyz=0.000175875481034 0 0 rpy=1.57201212277 0 -4.22293331334e-06 -> xyz=0.000175875481034 0 0 rpy=1.57201212277 1.047 -4.22293331334e-06
- joint shoulder_pan_joint: origin xyz=0 0 0.162509611124 rpy=0 0 3.14159265774 -> xyz=0 0 0.162509611124 rpy=0 0 0.785
- joint wrist_1_joint: origin xyz=-0.392424671078 0.000403177258085 0.13370723674 rpy=3.13857728923 -3.14158422042 3.14159213673 -> xyz=-0.392424671078 0.000403177258085 0.13370723674 rpy=3.13857728923 -3.14158422042 -1.047
- joint wrist_2_joint: origin xyz=-3.59538768323e-05 -0.0997732519853 3.17373243326e-05 rpy=1.57047823229 0 -1.22657964634e-06 -> xyz=-3.59538768323e-05 -0.0997732519853 3.17373243326e-05 rpy=1.57047823229 1.571 -1.22657964634e-06
