Commit message: modifications for path generations and voxel verification

File: urdf/ur5e/ur5e.urdf (robot description, URDF)
Before this commit: robot ur5e, 11 links, 10 joints
Links:
- added link ee_probe; visual cylinder length=0.1 radius=0.005
- added link ee_probe_tip
Joints:
- added joint ee_probe_joint: type fixed, parent ee_link, child ee_probe, origin xyz=0.05 0 0 rpy=0 1.57 0
- added joint ee_probe_tip_joint: type fixed, parent ee_probe, child ee_probe_tip, origin xyz=0 0 0.07 rpy=0 0 0

File: urdf/ur5e/ur5e_cart.urdf (robot description, URDF)
Before this commit: robot ur5e, 15 links, 14 joints
Links:
- link ee_probe: geometry visual cylinder length=0.1 radius=0.005
Joints:
- joint elbow_joint: origin xyz=-0.425282422158 0 0 rpy=3.14087106174 3.14130791395 -1.047 -> xyz=-0.425282422158 0 0 rpy=3.14087106174 3.14130791395 -3.1415908958
- joint shoulder_lift_joint: origin xyz=0.000175875481034 0 0 rpy=1.57201212277 1.047 -4.22293331334e-06 -> xyz=0.000175875481034 0 0 rpy=1.57201212277 0 -4.22293331334e-06
- joint shoulder_pan_joint: origin xyz=0 0 0.162509611124 rpy=0 0 0.785 -> xyz=0 0 0.162509611124 rpy=0 0 3.14159265774
- joint wrist_1_joint: origin xyz=-0.392424671078 0.000403177258085 0.13370723674 rpy=3.13857728923 -3.14158422042 -1.047 -> xyz=-0.392424671078 0.000403177258085 0.13370723674 rpy=3.13857728923 -3.14158422042 3.14159213673
- joint wrist_2_joint: origin xyz=-3.59538768323e-05 -0.0997732519853 3.17373243326e-05 rpy=1.57047823229 1.571 -1.22657964634e-06 -> xyz=-3.59538768323e-05 -0.0997732519853 3.17373243326e-05 rpy=1.57047823229 0 -1.22657964634e-06

Commit message: working with path interpolation

File: urdf/ur5e/ur5e.urdf (robot description, URDF)
Before this commit: robot ur5e, 13 links, 12 joints
Links:
- link ee_probe: geometry visual cylinder length=0.225 radius=0.005
Joints:
- joint ee_probe_joint: origin xyz=0.05 0 0 rpy=0 1.57 0 -> xyz=0.1125 0 0 rpy=0 1.57 0

Commit message: added fake gripper to urdf. adjusted joint interpolation. added self collision checking to trajectory generation

File: urdf/ur5e/ur5e.urdf (robot description, URDF)
Before this commit: robot ur5e, 13 links, 12 joints
Links:
- removed link ee_probe
- added link gripper_link; collision box size=0.06 0.06 0.2; visual box size=0.06 0.06 0.2
Joints:
- joint ee_probe_joint: child ee_probe -> gripper_link; origin xyz=0.1125 0 0 rpy=0 1.57 0 -> xyz=0.21 0 0 rpy=0 1.57 0
- joint ee_probe_tip_joint: origin xyz=0 0 0.07 rpy=0 0 0 -> xyz=-0.02 0 0 rpy=0 0 0; parent ee_probe -> gripper_link

Commit message: generating a voxelized volume instead of voxelized mesh of a parallelepiped. need to verify hole in path generation

File: urdf/ur5e/ur5e.urdf (robot description, URDF)
Before this commit: robot ur5e, 13 links, 12 joints
Links:
- removed link ee_probe_tip
Joints:
- removed joint ee_probe_joint
- removed joint ee_probe_tip_joint
- added joint gripper_joint: type fixed, parent tool0, child gripper_link, origin xyz=0 0 0.215 rpy=0 0 0

Commit message: refining trajectory generation, limiting target orientations to have minimal yaw rotation, adding doc strings

File: urdf/ur5e/ur5e.urdf (robot description, URDF)
Before this commit: robot ur5e, 12 links, 11 joints
Links:
- link gripper_link: geometry collision box size=0.12 0.12 0.2; visual box size=0.12 0.12 0.2
