Commit message: adds collision objects to prismatic joints -> prevents gaps in prismatic joint extension

File: manipulator_codesign/urdf/robots/nsga2_seeds/gen_seed_0.urdf (robot description, URDF)
Before this commit: robot NSGA_robot_balanced, 16 links, 15 joints
Links:
- link link3: geometry collision cylinder length=0.35859096102358173 radius=0.05; visual cylinder length=0.35859096102358173 radius=0.05
- link link4: geometry collision cylinder length=0.7416494040066779 radius=0.05; visual cylinder length=0.7416494040066779 radius=0.05
Joints:
- joint joint0: limit lower=-6.283185307179586 upper=6.283185307179586 effort=10 velocity=1 -> lower=-3.14 upper=3.14 effort=10 velocity=1
- joint joint1: limit lower=-6.283185307179586 upper=6.283185307179586 effort=10 velocity=1 -> lower=-3.14 upper=3.14 effort=10 velocity=1
- joint joint2: limit lower=-6.283185307179586 upper=6.283185307179586 effort=10 velocity=1 -> lower=-3.14 upper=3.14 effort=10 velocity=1
- joint joint3: limit lower=-0.5 upper=0.5 effort=10 velocity=1 -> lower=0 upper=0.3475909610235817 effort=10 velocity=1; origin xyz=0 0 0.4025909610235817 rpy=0 0 0 -> xyz=0 0 0.061 rpy=0 0 0
- joint joint4: limit lower=-6.283185307179586 upper=6.283185307179586 effort=10 velocity=1 -> lower=-3.14 upper=3.14 effort=10 velocity=1; origin xyz=0 0 0.38830290037953324 rpy=0 0 0 -> xyz=0 0 0.35859096102358173 rpy=0 0 0
- joint joint5: limit lower=-6.283185307179586 upper=6.283185307179586 effort=10 velocity=1 -> lower=-3.14 upper=3.14 effort=10 velocity=1; origin xyz=0 0 0.6575749836629056 rpy=0 0 0 -> xyz=0 0 0.7416494040066779 rpy=0 0 0
- joint joint6: limit lower=-6.283185307179586 upper=6.283185307179586 effort=10 velocity=1 -> lower=-3.14 upper=3.14 effort=10 velocity=1
- joint joint_viz4: origin xyz=0 0 0.38830290037953324 rpy=0 0 0 -> xyz=0 0 0.35859096102358173 rpy=0 0 0
- joint joint_viz5: origin xyz=0 0 0.6575749836629056 rpy=0 0 0 -> xyz=0 0 0.7416494040066779 rpy=0 0 0

File: manipulator_codesign/urdf/robots/nsga2_seeds/gen_seed_1.urdf (robot description, URDF)
Before this commit: robot test_robot, 16 links, 15 joints
Links:
- link link2: geometry collision cylinder length=0.461 radius=0.05; visual cylinder length=0.461 radius=0.05
Joints:
- joint joint2: limit lower=-0.5 upper=0.5 effort=10 velocity=1 -> lower=0 upper=0.45 effort=10 velocity=1; origin xyz=0 0 0.5 rpy=0 0 0 -> xyz=0 0 0.061 rpy=0 0 0
- joint joint3: origin xyz=0 0 0.3 rpy=0 0 0 -> xyz=0 0 0.461 rpy=0 0 0
- joint joint_viz3: origin xyz=0 0 0.3 rpy=0 0 0 -> xyz=0 0 0.461 rpy=0 0 0

File: manipulator_codesign/urdf/robots/nsga2_seeds/gen_seed_2.urdf (robot description, URDF)
Before this commit: robot test_robot, 15 links, 14 joints
Links:
- added link link0_fixed, mass 1.0; collision box size=0.1 1.1 0.05; visual box size=0.1 1.1 0.05
- link link2: geometry collision cylinder length=0.261 radius=0.05; visual cylinder length=0.261 radius=0.05
Joints:
- added joint joint0_fixed: type fixed, parent base_link, child link0_fixed, origin xyz=0 0 0.125 rpy=0 0 0
- joint joint0: origin xyz=0 0 0.125 rpy=0 0 0 -> xyz=0 0 0 rpy=0 0 0; parent base_link -> link0_fixed
- joint joint2: limit lower=-0.5 upper=0.5 effort=10 velocity=1 -> lower=0 upper=0.25 effort=10 velocity=1; origin xyz=0 0 0.3 rpy=0 0 0 -> xyz=0 0 0.061 rpy=0 0 0
- joint joint3: origin xyz=0 0 0.3 rpy=0 0 0 -> xyz=0 0 0.261 rpy=0 0 0
- joint joint_viz3: origin xyz=0 0 0.3 rpy=0 0 0 -> xyz=0 0 0.261 rpy=0 0 0

File: manipulator_codesign/urdf/robots/nsga2_seeds/gen_seed_3.urdf (robot description, URDF)
Before this commit: robot test_robot, 13 links, 12 joints
Links:
- added link link0_fixed, mass 1.0; collision box size=0.1 1.1 0.05; visual box size=0.1 1.1 0.05
- link link2: geometry collision cylinder length=0.261 radius=0.05; visual cylinder length=0.261 radius=0.05
Joints:
- added joint joint0_fixed: type fixed, parent base_link, child link0_fixed, origin xyz=0 0 0.125 rpy=0 0 0
- joint joint0: origin xyz=0 0 0.125 rpy=0 0 0 -> xyz=0 0 0 rpy=0 0 0; parent base_link -> link0_fixed
- joint joint2: limit lower=-0.5 upper=0.5 effort=10 velocity=1 -> lower=0 upper=0.25 effort=10 velocity=1; origin xyz=0 0 0.3 rpy=0 0 0 -> xyz=0 0 0.061 rpy=0 0 0
- joint joint3: origin xyz=0 0 0.3 rpy=0 0 0 -> xyz=0 0 0.261 rpy=0 0 0
- joint joint_viz3: origin xyz=0 0 0.3 rpy=0 0 0 -> xyz=0 0 0.261 rpy=0 0 0

File: manipulator_codesign/urdf/robots/nsga2_seeds/gen_seed_4.urdf (robot description, URDF)
Before this commit: robot test_robot, 14 links, 13 joints
Links:
- link link1: geometry collision cylinder length=0.461 radius=0.05; visual cylinder length=0.461 radius=0.05
Joints:
- joint joint1: limit lower=-0.5 upper=0.5 effort=10 velocity=1 -> lower=0 upper=0.45 effort=10 velocity=1; origin xyz=0 0 0.5 rpy=0 0 0 -> xyz=0 0 0.061 rpy=0 0 0
- joint joint2: origin xyz=0 0 0.3 rpy=0 0 0 -> xyz=0 0 0.461 rpy=0 0 0
- joint joint_viz2: origin xyz=0 0 0.3 rpy=0 0 0 -> xyz=0 0 0.461 rpy=0 0 0

File: manipulator_codesign/urdf/robots/nsga2_seeds/gen_seed_5.urdf (robot description, URDF)
Before this commit: robot test_robot, 16 links, 15 joints
Links:
- link link3: geometry collision cylinder length=0.261 radius=0.05; visual cylinder length=0.261 radius=0.05
Joints:
- joint joint3: limit lower=-0.5 upper=0.5 effort=10 velocity=1 -> lower=0 upper=0.25 effort=10 velocity=1; origin xyz=0 0 0.3 rpy=0 0 0 -> xyz=0 0 0.061 rpy=0 0 0
- joint joint4: origin xyz=0 0 0.4 rpy=0 0 0 -> xyz=0 0 0.261 rpy=0 0 0
- joint joint_viz4: origin xyz=0 0 0.4 rpy=0 0 0 -> xyz=0 0 0.261 rpy=0 0 0

File: manipulator_codesign/urdf/robots/nsga2_seeds/gen_seed_6.urdf (robot description, URDF)
Before this commit: robot test_robot, 15 links, 14 joints
Links:
- removed link joint_viz_link0
- removed link joint_viz_link1
- removed link joint_viz_link5
- removed link joint_viz_link6
- added link joint_viz_link2, mass 0.0; visual cylinder length=0.125 radius=0.06
- added link joint_viz_link3, mass 0.0; visual cylinder length=0.125 radius=0.06
- added link link0_fixed, mass 1.0; collision box size=1.1 0.1 0.05; visual box size=1.1 0.1 0.05
- added link link1_fixed, mass 1.0; collision box size=0.1 1.1 0.05; visual box size=0.1 1.1 0.05
- added link sph_link_x_1, mass 0.001; visual sphere radius=0.1
- added link sph_link_y_1, mass 0.001; visual sphere radius=0.1
- added link sph_link_z_1, mass 0.001; visual sphere radius=0.1
- link link0: geometry collision cylinder length=0.05 radius=0.05; visual cylinder length=0.05 radius=0.05
- link link1: geometry collision cylinder length=0.05 radius=0.05; visual cylinder length=0.05 radius=0.05
- link link2: geometry collision cylinder length=0.75 radius=0.05; visual cylinder length=0.75 radius=0.05
- link link3: geometry collision cylinder length=0.5 radius=0.05; visual cylinder length=0.5 radius=0.05
- link link4: geometry collision cylinder length=0.5 radius=0.05; visual cylinder length=0.5 radius=0.05
- link link5: geometry collision cylinder length=0.461 radius=0.05; visual cylinder length=0.461 radius=0.05
- link link6: geometry collision cylinder length=0.1 radius=0.05; visual cylinder length=0.1 radius=0.05
Joints:
- removed joint joint_viz0
- removed joint joint_viz1
- removed joint joint_viz5
- removed joint joint_viz6
- added joint joint0_fixed: type fixed, parent base_link, child link0_fixed, origin xyz=0 0 0.125 rpy=0 0 0
- added joint joint1_fixed: type fixed, parent link0, child link1_fixed, origin xyz=0 0 0.05 rpy=0 0 0
- added joint joint_viz2: type fixed, parent link1, child joint_viz_link2, origin xyz=0 0 0.05 rpy=0 0 0
- added joint joint_viz3: type fixed, parent link2, child joint_viz_link3, origin xyz=0 0 0.75 rpy=0 0 0
- added joint sph_joint_x_1: type revolute, parent link5, child sph_link_x_1, origin xyz=0 0 0.461 rpy=0 0 0, axis 1 0 0, limit lower=-3.14 upper=3.14 effort=10 velocity=1
- added joint sph_joint_y_1: type revolute, parent sph_link_x_1, child sph_link_y_1, origin xyz=0 0 0 rpy=0 0 0, axis 0 1 0, limit lower=-3.14 upper=3.14 effort=10 velocity=1
- added joint sph_joint_z_1: type revolute, parent sph_link_y_1, child sph_link_z_1, origin xyz=0 0 0 rpy=0 0 0, axis 0 0 1, limit lower=-3.14 upper=3.14 effort=10 velocity=1
- joint joint0: axis 0 0 1 -> 1 0 0; limit lower=-3.14 upper=3.14 effort=10 velocity=1 -> lower=-0.5 upper=0.5 effort=10 velocity=1; origin xyz=0 0 0.125 rpy=0 0 0 -> xyz=0 0 0 rpy=0 0 0; parent base_link -> link0_fixed; type revolute -> prismatic
- joint joint1: axis 1 0 0 -> 0 1 0; limit lower=-3.14 upper=3.14 effort=10 velocity=1 -> lower=-0.5 upper=0.5 effort=10 velocity=1; origin xyz=0 0 0.4 rpy=0 0 0 -> xyz=0 0 0 rpy=0 0 0; parent link0 -> link1_fixed; type revolute -> prismatic
- joint joint2: axis 0 1 0 -> 0 0 1; limit lower=-0.5 upper=0.5 effort=10 velocity=1 -> lower=-3.14 upper=3.14 effort=10 velocity=1; origin xyz=0 0 0.5 rpy=0 0 0 -> xyz=0 0 0.05 rpy=0 0 0; type prismatic -> revolute
- joint joint3: axis 0 0 1 -> 1 0 0; limit lower=-0.5 upper=0.5 effort=10 velocity=1 -> lower=-3.14 upper=3.14 effort=10 velocity=1; origin xyz=0 0 0.5 rpy=0 0 0 -> xyz=0 0 0.75 rpy=0 0 0; type prismatic -> revolute
- joint joint4: axis 0 0 1 -> 0 1 0; origin xyz=0 0 0.4 rpy=0 0 0 -> xyz=0 0 0.5 rpy=0 0 0
- joint joint5: axis 1 0 0 -> 0 0 1; limit lower=-3.14 upper=3.14 effort=10 velocity=1 -> lower=0 upper=0.45 effort=10 velocity=1; origin xyz=0 0 0.1 rpy=0 0 0 -> xyz=0 0 0.061 rpy=0 0 0; type revolute -> prismatic
- joint joint6: axis 0 1 0 -> (none); limit lower=-3.14 upper=3.14 effort=10 velocity=1 -> (none); origin xyz=0 0 0.4 rpy=0 0 0 -> xyz=0 0 0 rpy=0 0 0; parent link5 -> sph_link_z_1; type revolute -> fixed
- joint joint_viz4: origin xyz=0 0 0.4 rpy=0 0 0 -> xyz=0 0 0.5 rpy=0 0 0
- joint probe_joint: origin xyz=0 0 0.4 rpy=0 0 0 -> xyz=0 0 0.1 rpy=0 0 0

File: manipulator_codesign/urdf/robots/nsga2_seeds/gen_seed_7.urdf (robot description, URDF)
Before this commit: robot test_robot, 13 links, 12 joints
Links:
- removed link joint_viz_link0
- removed link joint_viz_link1
- added link joint_viz_link2, mass 0.0; visual cylinder length=0.125 radius=0.06
- added link link0_fixed, mass 1.0; collision box size=1.1 0.1 0.05; visual box size=1.1 0.1 0.05
- added link link1_fixed, mass 1.0; collision box size=0.1 1.1 0.05; visual box size=0.1 1.1 0.05
- added link link5, mass 1.0; collision cylinder length=0.5609999999999999 radius=0.05; visual cylinder length=0.5609999999999999 radius=0.05
- link link0: geometry collision cylinder length=0.05 radius=0.05; visual cylinder length=0.05 radius=0.05
- link link1: geometry collision cylinder length=0.05 radius=0.05; visual cylinder length=0.05 radius=0.05
- link link2: geometry collision cylinder length=0.75 radius=0.05; visual cylinder length=0.75 radius=0.05
- link link3: geometry collision cylinder length=0.711 radius=0.05; visual cylinder length=0.711 radius=0.05
- link link4: geometry collision cylinder length=0.6 radius=0.05; visual cylinder length=0.6 radius=0.05
Joints:
- removed joint joint_viz0
- removed joint joint_viz1
- added joint joint0_fixed: type fixed, parent base_link, child link0_fixed, origin xyz=0 0 0.125 rpy=0 0 0
- added joint joint1_fixed: type fixed, parent link0, child link1_fixed, origin xyz=0 0 0.05 rpy=0 0 0
- added joint joint5: type prismatic, parent link4, child link5, origin xyz=0 0 0.061 rpy=0 0 0, axis 0 0 1, limit lower=0 upper=0.5499999999999999 effort=10 velocity=1
- added joint joint_viz2: type fixed, parent link1, child joint_viz_link2, origin xyz=0 0 0.05 rpy=0 0 0
- joint joint0: axis 0 0 1 -> 1 0 0; limit lower=-3.14 upper=3.14 effort=10 velocity=1 -> lower=-0.5 upper=0.5 effort=10 velocity=1; origin xyz=0 0 0.125 rpy=0 0 0 -> xyz=0 0 0 rpy=0 0 0; parent base_link -> link0_fixed; type revolute -> prismatic
- joint joint1: axis 1 0 0 -> 0 1 0; limit lower=-3.14 upper=3.14 effort=10 velocity=1 -> lower=-0.5 upper=0.5 effort=10 velocity=1; origin xyz=0 0 0.4 rpy=0 0 0 -> xyz=0 0 0 rpy=0 0 0; parent link0 -> link1_fixed; type revolute -> prismatic
- joint joint2: axis 0 1 0 -> 1 0 0; limit lower=-0.5 upper=0.5 effort=10 velocity=1 -> lower=-3.14 upper=3.14 effort=10 velocity=1; origin xyz=0 0 0.5 rpy=0 0 0 -> xyz=0 0 0.05 rpy=0 0 0; type prismatic -> revolute
- joint joint3: limit lower=-0.5 upper=0.5 effort=10 velocity=1 -> lower=0 upper=0.7 effort=10 velocity=1; origin xyz=0 0 0.6 rpy=0 0 0 -> xyz=0 0 0.061 rpy=0 0 0
- joint probe_joint: origin xyz=0 0 0.1 rpy=0 0 0 -> xyz=0 0 0.5609999999999999 rpy=0 0 0; parent link4 -> link5
- joint sph_joint_x_1: origin xyz=0 0 0.6 rpy=0 0 0 -> xyz=0 0 0.711 rpy=0 0 0

File: manipulator_codesign/urdf/robots/nsga2_seeds/gen_seed_9.urdf (robot description, URDF)
Before this commit: robot test_robot, 15 links, 14 joints
Links:
- removed link joint_viz_link0
- removed link joint_viz_link2
- removed link joint_viz_link3
- removed link link5
- added link sph_link_x_2, mass 0.001; visual sphere radius=0.1
- added link sph_link_x_3, mass 0.001; visual sphere radius=0.1
- added link sph_link_y_2, mass 0.001; visual sphere radius=0.1
- added link sph_link_y_3, mass 0.001; visual sphere radius=0.1
- added link sph_link_z_2, mass 0.001; visual sphere radius=0.1
- added link sph_link_z_3, mass 0.001; visual sphere radius=0.1
- link link2: geometry collision cylinder length=0.5 radius=0.05; visual cylinder length=0.5 radius=0.05
- link link3: geometry collision cylinder length=0.461 radius=0.05; visual cylinder length=0.461 radius=0.05
- link link4: geometry collision cylinder length=0.4 radius=0.05; visual cylinder length=0.4 radius=0.05
Joints:
- removed joint joint5
- removed joint joint_viz0
- removed joint joint_viz2
- removed joint joint_viz3
- added joint sph_joint_x_2: type revolute, parent link1, child sph_link_x_2, origin xyz=0 0 0.711 rpy=0 0 0, axis 1 0 0, limit lower=-3.14 upper=3.14 effort=10 velocity=1
- added joint sph_joint_x_3: type revolute, parent link3, child sph_link_x_3, origin xyz=0 0 0.461 rpy=0 0 0, axis 1 0 0, limit lower=-3.14 upper=3.14 effort=10 velocity=1
- added joint sph_joint_y_2: type revolute, parent sph_link_x_2, child sph_link_y_2, origin xyz=0 0 0 rpy=0 0 0, axis 0 1 0, limit lower=-3.14 upper=3.14 effort=10 velocity=1
- added joint sph_joint_y_3: type revolute, parent sph_link_x_3, child sph_link_y_3, origin xyz=0 0 0 rpy=0 0 0, axis 0 1 0, limit lower=-3.14 upper=3.14 effort=10 velocity=1
- added joint sph_joint_z_2: type revolute, parent sph_link_y_2, child sph_link_z_2, origin xyz=0 0 0 rpy=0 0 0, axis 0 0 1, limit lower=-3.14 upper=3.14 effort=10 velocity=1
- added joint sph_joint_z_3: type revolute, parent sph_link_y_3, child sph_link_z_3, origin xyz=0 0 0 rpy=0 0 0, axis 0 0 1, limit lower=-3.14 upper=3.14 effort=10 velocity=1
- joint joint0: axis 1 0 0 -> (none); limit lower=-3.14 upper=3.14 effort=10 velocity=1 -> (none); origin xyz=0 0 0.125 rpy=0 0 0 -> xyz=0 0 0 rpy=0 0 0; parent base_link -> sph_link_z_1; type revolute -> fixed
- joint joint2: axis 0 0 1 -> (none); limit lower=-3.14 upper=3.14 effort=10 velocity=1 -> (none); origin xyz=0 0 0.711 rpy=0 0 0 -> xyz=0 0 0 rpy=0 0 0; parent link1 -> sph_link_z_2; type revolute -> fixed
- joint joint3: axis 0 1 0 -> 0 0 1; limit lower=-3.14 upper=3.14 effort=10 velocity=1 -> lower=0 upper=0.45 effort=10 velocity=1; origin xyz=0 0 0.05 rpy=0 0 0 -> xyz=0 0 0.061 rpy=0 0 0; type revolute -> prismatic
- joint joint4: axis 0 0 1 -> (none); limit lower=0 upper=0.45 effort=10 velocity=1 -> (none); origin xyz=0 0 0.061 rpy=0 0 0 -> xyz=0 0 0 rpy=0 0 0; parent link3 -> sph_link_z_3; type prismatic -> fixed
- joint probe_joint: origin xyz=0 0 0.1 rpy=0 0 0 -> xyz=0 0 0.4 rpy=0 0 0; parent link5 -> link4
- joint sph_joint_x_1: origin xyz=0 0 0.461 rpy=0 0 0 -> xyz=0 0 0.125 rpy=0 0 0; parent link4 -> base_link

Commit message: repo cleanup, benchmark setup, env staging

File: manipulator_codesign/urdf/robots/nsga2_seeds/gen_seed_0.urdf (robot description, URDF)
Before this commit: robot test_robot, 16 links, 15 joints
Links:
- removed link joint_viz_link6
- removed link link6
- added link joint_viz_link3, mass 0.0; visual cylinder length=0.05 radius=0.03
- link base_link: geometry visual box size=0.75 0.25 0.25
- link joint_viz_link0: geometry visual cylinder length=0.05 radius=0.03
- link joint_viz_link1: geometry visual cylinder length=0.05 radius=0.03
- link joint_viz_link2: geometry visual cylinder length=0.05 radius=0.03
- link joint_viz_link4: geometry visual cylinder length=0.05 radius=0.03
- link joint_viz_link5: geometry visual cylinder length=0.05 radius=0.03
- link link0: geometry collision cylinder length=0.185 radius=0.025; visual cylinder length=0.185 radius=0.025
- link link1: geometry collision cylinder length=0.185 radius=0.025; visual cylinder length=0.185 radius=0.025
- link link2: geometry collision cylinder length=0.185 radius=0.025; visual cylinder length=0.185 radius=0.025
- link link3: geometry collision cylinder length=0.185 radius=0.025; visual cylinder length=0.185 radius=0.025
- link link4: geometry collision cylinder length=0.185 radius=0.025; visual cylinder length=0.185 radius=0.025
- link link5: geometry collision cylinder length=0.185 radius=0.025; visual cylinder length=0.185 radius=0.025
Joints:
- removed joint joint6
- removed joint joint_viz6
- added joint joint_viz3: type fixed, parent link2, child joint_viz_link3, origin xyz=0 0 0.185 rpy=0 0 0
- joint joint1: axis 1 0 0 -> 0 1 0; origin xyz=0 0 0.4453456610645649 rpy=0 0 0 -> xyz=0 0 0.185 rpy=0 0 0
- joint joint2: axis 0 1 0 -> 1 0 0; origin xyz=0 0 0.26184065228893466 rpy=0 0 0 -> xyz=0 0 0.185 rpy=0 0 0
- joint joint3: limit lower=0 upper=0.3475909610235817 effort=10 velocity=1 -> lower=-3.14 upper=3.14 effort=10 velocity=1; origin xyz=0 0 0.061 rpy=0 0 0 -> xyz=0 0 0.185 rpy=0 0 0; type prismatic -> revolute
- joint joint4: axis 1 0 0 -> 0 1 0; origin xyz=0 0 0.35859096102358173 rpy=0 0 0 -> xyz=0 0 0.185 rpy=0 0 0
- joint joint5: origin xyz=0 0 0.7416494040066779 rpy=0 0 0 -> xyz=0 0 0.185 rpy=0 0 0
- joint joint_viz1: origin xyz=0 0 0.4453456610645649 rpy=0 0 0 -> xyz=0 0 0.185 rpy=0 0 0
- joint joint_viz2: origin xyz=0 0 0.26184065228893466 rpy=0 0 0 -> xyz=0 0 0.185 rpy=0 0 0
- joint joint_viz4: origin xyz=0 0 0.35859096102358173 rpy=0 0 0 -> xyz=0 0 0.185 rpy=0 0 0
- joint joint_viz5: origin xyz=0 0 0.7416494040066779 rpy=0 0 0 -> xyz=0 0 0.185 rpy=0 0 0
- joint probe_joint: origin xyz=0 0 0.1 rpy=0 0 0 -> xyz=0 0 0.185 rpy=0 0 0; parent link6 -> link5

File: manipulator_codesign/urdf/robots/nsga2_seeds/gen_seed_1.urdf (robot description, URDF)
Before this commit: robot test_robot, 16 links, 15 joints
Links:
- removed link sph_link_x_1
- removed link sph_link_y_1
- removed link sph_link_z_1
- added link joint_viz_link0, mass 0.0; visual cylinder length=0.05 radius=0.03
- added link joint_viz_link2, mass 0.0; visual cylinder length=0.05 radius=0.03
- added link joint_viz_link6, mass 0.0; visual cylinder length=0.05 radius=0.03
- added link link6, mass 1.0; collision cylinder length=0.185 radius=0.025; visual cylinder length=0.185 radius=0.025
- link base_link: geometry visual box size=0.75 0.25 0.25
- link joint_viz_link1: geometry visual cylinder length=0.05 radius=0.03
- link joint_viz_link3: geometry visual cylinder length=0.05 radius=0.03
- link joint_viz_link4: geometry visual cylinder length=0.05 radius=0.03
- link joint_viz_link5: geometry visual cylinder length=0.05 radius=0.03
- link link0: geometry collision cylinder length=0.185 radius=0.025; visual cylinder length=0.185 radius=0.025
- link link1: geometry collision cylinder length=0.185 radius=0.025; visual cylinder length=0.185 radius=0.025
- link link2: geometry collision cylinder length=0.185 radius=0.025; visual cylinder length=0.185 radius=0.025
- link link3: geometry collision cylinder length=0.185 radius=0.025; visual cylinder length=0.185 radius=0.025
- link link4: geometry collision cylinder length=0.185 radius=0.025; visual cylinder length=0.185 radius=0.025
- link link5: geometry collision cylinder length=0.185 radius=0.025; visual cylinder length=0.185 radius=0.025
Joints:
- removed joint sph_joint_x_1
- removed joint sph_joint_y_1
- removed joint sph_joint_z_1
- added joint joint6: type revolute, parent link5, child link6, origin xyz=0 0 0.185 rpy=0 0 0, axis 0 1 0, limit lower=-3.14 upper=3.14 effort=10 velocity=1
- added joint joint_viz0: type fixed, parent base_link, child joint_viz_link0, origin xyz=0 0 0.125 rpy=0 0 0
- added joint joint_viz2: type fixed, parent link1, child joint_viz_link2, origin xyz=0 0 0.185 rpy=0 0 0
- added joint joint_viz6: type fixed, parent link5, child joint_viz_link6, origin xyz=0 0 0.185 rpy=0 0 0
- joint joint0: axis (none) -> 0 0 1; limit (none) -> lower=-3.14 upper=3.14 effort=10 velocity=1; origin xyz=0 0 0 rpy=0 0 0 -> xyz=0 0 0.125 rpy=0 0 0; parent sph_link_z_1 -> base_link; type fixed -> revolute
- joint joint1: axis 1 0 0 -> 0 1 0; origin xyz=0 0 0.5 rpy=0 0 0 -> xyz=0 0 0.185 rpy=0 0 0
- joint joint2: axis 0 0 1 -> 1 0 0; limit lower=0 upper=0.45 effort=10 velocity=1 -> lower=-3.14 upper=3.14 effort=10 velocity=1; origin xyz=0 0 0.061 rpy=0 0 0 -> xyz=0 0 0.185 rpy=0 0 0; type prismatic -> revolute
- joint joint3: axis 1 0 0 -> 0 0 1; origin xyz=0 0 0.461 rpy=0 0 0 -> xyz=0 0 0.185 rpy=0 0 0
- joint joint4: axis 1 0 0 -> 0 1 0; origin xyz=0 0 0.5 rpy=0 0 0 -> xyz=0 0 0.185 rpy=0 0 0
- joint joint5: axis 0 1 0 -> 1 0 0; origin xyz=0 0 0.35 rpy=0 0 0 -> xyz=0 0 0.185 rpy=0 0 0
- joint joint_viz1: origin xyz=0 0 0.5 rpy=0 0 0 -> xyz=0 0 0.185 rpy=0 0 0
- joint joint_viz3: origin xyz=0 0 0.461 rpy=0 0 0 -> xyz=0 0 0.185 rpy=0 0 0
- joint joint_viz4: origin xyz=0 0 0.5 rpy=0 0 0 -> xyz=0 0 0.185 rpy=0 0 0
- joint joint_viz5: origin xyz=0 0 0.35 rpy=0 0 0 -> xyz=0 0 0.185 rpy=0 0 0
- joint probe_joint: origin xyz=0 0 0.1 rpy=0 0 0 -> xyz=0 0 0.185 rpy=0 0 0; parent link5 -> link6
